File: Xbox-Charge.kicad_sch (KiCad schematic)
At the start: 91 parts, among them J1 Conn_01x04_Pin, J2 Conn_01x04_Pin, Q1 CSD17551Q3A, Q2 CSD17551Q3A, Q3 CSD17551Q3A, Q4 CSD17551Q3A, Q5 CSD25402Q3A, U1 TPS25750, U2 BQ25713RSNR, U3 CAT24C512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

Commit message: Cleaned up schematic and split BQ25713 circuit off to a second sheet
Parts:
- R8: value 750K -> 300K
- R9: value 250K -> 100K
Other:
- added sheet BQ25713 (BQ25713.kicad_sch)
- moved on the sheet: BT1, C1, C10, C11, C12, C13, C14, C15, C16, C17, C18, C19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
